File: kikad/ambient/ambient.kicad_pcb (KiCad board)
At the start: 2 copper layers, 35 parts, among them J1 5V DC, J2 FPC 01x10 Female, SW1 Reset, SW2 Next, SW3 Select, SW4 Modify, U1 ATmega328P-PU, Y1 16 MHz

Commit message: fixes
Parts:
- added C12: 0.1u, Capacitor_SMD:C_1206_3216Metric, F.Cu at (67.3, 71.3)
- added C13: 0.1u, Capacitor_SMD:C_1206_3216Metric, F.Cu at (72.9, 71.3)
- added C14: 0.1u, Capacitor_SMD:C_1206_3216Metric, F.Cu at (67.3, 74.7)
- added C15: 0.1u, Capacitor_SMD:C_1206_3216Metric, F.Cu at (90.5, 59.6)
- added R12: 4.7k, Resistor_SMD:R_0805_2012Metric, F.Cu at (72.3, 74.5)
- added R13: 4.7k, Resistor_SMD:R_0805_2012Metric, F.Cu at (66.6, 77.8)
- added R14: 4.7k, Resistor_SMD:R_0805_2012Metric, F.Cu at (77.9, 71.1)
- added R15: 4.7k, Resistor_SMD:R_0805_2012Metric, F.Cu at (71.1, 77.8)
- added R16: 4.7k, Resistor_SMD:R_0805_2012Metric, F.Cu at (89.8, 62.7)
- added R17: 4.7k, Resistor_SMD:R_0805_2012Metric, F.Cu at (77.9, 74.1)
- added U2: AT24C256, Package_DIP:DIP-8_W7.62mm_LongPads, F.Cu at (54.8, 60.0)
- added U3: AT24C256, Package_DIP:DIP-8_W7.62mm_LongPads, F.Cu at (54.8, 71.7)
- added U4: AT24C256, Package_DIP:DIP-8_W7.62mm_LongPads, F.Cu at (66.4, 60.0)
- added U5: AT24C256, Package_DIP:DIP-8_W7.62mm_LongPads, F.Cu at (78.0, 60.0)
- moved SW1 25.5 mm to (78.7, 50.8)
Connections:
- U1 pad 27: Net-(U1-Pad27) -> SDA
- U1 pad 28: Net-(U1-Pad28) -> SCL

Commit message: draft +3
Parts:
- added C16: 0.1u, Capacitor_SMD:C_1206_3216Metric, F.Cu at (113.5, 81.4)
- added C17: 0.1u, Capacitor_SMD:C_1206_3216Metric, F.Cu at (130.3, 75.4)
- added C18: 0.1u, Capacitor_SMD:C_1206_3216Metric, F.Cu at (121.0, 77.1)
- added C19: 0.1u, Capacitor_SMD:C_1206_3216Metric, F.Cu at (119.1, 81.4)
- added D3: 1N4735A, Diode_THT:D_DO-41_SOD81_P10.16mm_Horizontal, F.Cu at (39.4, 73.7)
- added D4: 1N4735A, Diode_THT:D_DO-41_SOD81_P10.16mm_Horizontal, F.Cu at (15.2, 73.7)
- added D5: 1N4735A, Diode_THT:D_DO-41_SOD81_P10.16mm_Horizontal, F.Cu at (15.2, 61.0)
- added DD1: WS2812B, LED_SMD:LED_WS2812B_PLCC4_5.0x5.0mm_P3.2mm, F.Cu at (120.6, 86.6)
- added DD2: WS2812B, LED_SMD:LED_WS2812B_PLCC4_5.0x5.0mm_P3.2mm, F.Cu at (129.0, 86.6)
- added J3: LED Array, Connector_PinHeader_2.54mm:PinHeader_1x03_P2.54mm_Vertical, F.Cu at (15.2, 64.8)
- added Q1: 2N3904, Package_TO_SOT_THT:TO-92_Inline, F.Cu at (129.4, 71.1)
- added R18: 1k, Resistor_SMD:R_0805_2012Metric, F.Cu at (129.7, 78.5)
- added R19: 470, Resistor_SMD:R_1206_3216Metric, F.Cu at (124.7, 80.4)
- added R20: 0.02, Resistor_SMD:R_2512_6332Metric, F.Cu at (106.3, 73.9)
- added R21: 0.02, Resistor_SMD:R_2512_6332Metric, F.Cu at (106.3, 78.8)
- added R22: 0.02, Resistor_SMD:R_2512_6332Metric, F.Cu at (129.5, 65.4)
- added R23: 0.02, Resistor_SMD:R_2512_6332Metric, F.Cu at (115.5, 69.7)
- moved R10 95.6 mm to (26.7, 26.7), turned to 90 degrees
- moved D1 94.7 mm to (26.7, 31.8), turned to 90 degrees
- moved C11 92.7 mm to (31.8, 16.7), turned to 270 degrees
- moved RV1 65.4 mm to (34.3, 30.5)
- moved J2 59.9 mm to (43.2, 19.1), turned to 180 degrees
- moved C5 51.6 mm to (19.1, 30.5)
- moved C6 51.5 mm to (19.1, 53.3)
- moved C3 44.8 mm to (56.2, 25.4), turned to 180 degrees
- moved SW1 41.6 mm to (93.0, 11.7)
- moved Y1 39.1 mm to (55.9, 29.8), turned to 180 degrees
- moved L1 38.9 mm to (19.1, 41.9), turned to 270 degrees
- moved U1 36.7 mm to (73.7, 36.8), turned to 270 degrees
- moved R1 33.2 mm to (51.8, 33.7)
- moved SW2 33.2 mm to (93.0, 20.2)
- moved SW3 32.9 mm to (103.5, 11.7)
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Connections:
- U1 pad 15: Net-(U1-Pad15) -> PREVIEW_ARRAY
- U1 pad 16: Net-(U1-Pad16) -> MAIN_ARRAY
- U1 pad 24: Net-(U1-Pad24) -> AMP_IN

Commit message: pcb draft
Parts:
- added  : MountingHole_3.2mm_M3, MountingHole:MountingHole_3.2mm_M3, F.Cu at (79.4, 63.5)
- added  : MountingHole_3.2mm_M3, MountingHole:MountingHole_3.2mm_M3, F.Cu at (59.7, 20.3)
- moved R19 104.1 mm to (28.6, 40.6), turned to 90 degrees
- moved Q1 99.9 mm to (34.3, 40.6)
- moved R18 97.1 mm to (40.6, 40.0), turned to 90 degrees
- moved R22 96.6 mm to (33.7, 52.7), turned to 270 degrees
- moved C18 91.5 mm to (35.6, 44.5), turned to 180 degrees
- moved   87.7 mm to (31.8, 71.1)
- moved C19 79.1 mm to (43.8, 57.1), turned to 90 degrees
- moved R23 78.0 mm to (39.4, 52.7), turned to 270 degrees
- moved SW1 76.9 mm to (41.9, 69.2)
- moved R11 75.7 mm to (55.2, 49.5)
- moved SW3 74.7 mm to (55.9, 69.2)
- moved DD1 74.0 mm to (52.7, 57.1), turned to 90 degrees
- moved R20 73.7 mm to (33.7, 61.6), turned to 270 degrees
- moved DD2 72.4 mm to (62.9, 57.1), turned to 90 degrees
- moved C7 71.6 mm to (38.1, 71.8), turned to 270 degrees
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Routing:
- net AMP_IN: track 0.00 -> 65.2 mm
- net GND: track 0.00 -> 40.6 mm, vias 0 -> 72
- net SDA: track 0.00 -> 24.9 mm
- net ARRAY_DIN: track 0.00 -> 20.4 mm
- net VCC: track 0.00 -> 17.7 mm
- net RESET: track 0.00 -> 15.8 mm
- net SELECT: track 0.00 -> 15.5 mm
- net NEXT: track 0.00 -> 15.5 mm
- net MODIFY: track 0.00 -> 15.5 mm
- net XTAL1: track 0.00 -> 13.5 mm
- net XTAL2: track 0.00 -> 12.0 mm
- net Net-(R5-Pad2): track 0.00 -> 10.3 mm
- net Net-(R15-Pad2): track 0.00 -> 9.90 mm
- net Net-(R7-Pad2): track 0.00 -> 9.76 mm
- net Net-(R3-Pad2): track 0.00 -> 9.76 mm
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- added copper zone on B.Cu, net +5V
- added copper zone on F.Cu, net +5V
- added copper zone on F.Cu, net AMP_IN
- added copper zone on B.Cu, net GND
- added copper zone on F.Cu, net GND
- added copper zone on F.Cu, net Net-(R20-Pad1)
Other:
- board outline added: 80 x 66 mm
- board text added: "+"

Commit message: pcb first version
Parts:
- Q1: footprint Package_TO_SOT_THT:TO-92_Inline -> Package_TO_SOT_THT:TO-92
- moved Y1 0.64 mm to (59.1, 31.1)
- moved C3 0.63 mm to (59.4, 26.7)
- moved C4 0.63 mm to (54.0, 26.7)
Routing:
- net VCC: track 17.7 -> 202.5 mm, vias 0 -> 6
- net SCL: track 0.00 -> 80.6 mm, vias 0 -> 6
- net SDA: track 24.9 -> 79.5 mm
- net RESET: track 15.8 -> 69.3 mm
- net SELECT: track 15.5 -> 58.6 mm, vias 0 -> 2
- net LCD_DB4: track 0.00 -> 38.8 mm, vias 0 -> 4
- net NEXT: track 15.5 -> 52.8 mm, vias 0 -> 2
- net LCD_EN: track 0.00 -> 25.2 mm
- net ARRAY_DIN: track 20.4 -> 45.2 mm
- net MODIFY: track 15.5 -> 37.9 mm, vias 0 -> 1
- net LCD_DB5: track 0.00 -> 19.7 mm, vias 0 -> 2
- net LCD_DB7: track 0.00 -> 17.1 mm
- net LCD_DB6: track 0.00 -> 16.4 mm, vias 0 -> 2
- net LCD_RS: track 0.00 -> 16.0 mm
- net PREVIEW_ARRAY: track 0.00 -> 13.0 mm, vias 0 -> 2
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- added copper zone on F.Cu, net VCC
Other:
- board text removed: "+"

Commit message: bug fixes, first version
Parts:
- moved C1 1.27 mm to (61.6, 49.5)
Routing:
- net VCC: track 202.5 -> 204.2 mm
Changed lines of the file:
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@@
     (thickness 1.6)
     (drawings 5)
-    (tracks 486)
+    (tracks 489)
     (zones 0)
     (modules 68)
@@
   )
   (module Capacitor_SMD:C_1206_3216Metric (layer F.Cu)
-    (at 60.325 49.53)
+    (at 61.595 49.53)
     (descr "Capacitor SMD 1206 (3216 Metric), square (rectangular) end terminal, IPC_7351 nominal, (Body size source: IPC-SM-782 page 76, https://www.pcb-3d.com/wordpress/wp-content/uploads/ipc-sm-782a_amendment_1_and_2.pdf), generated with kicad-footprint-generator")
     (tags capacitor)
@@
   (gr_line (start 93.98 13.97) (end 93.98 78.74) (layer Edge.Cuts) (width 0.05))
   (gr_line (start 13.97 13.97) (end 93.98 13.97) (layer Edge.Cuts) (width 0.05))
-  (via (at 59.055 53.34) (size 0.8) (drill 0.4) (layers F.Cu B.Cu) (net 10))
-  (via (at 57.785 53.34) (size 0.8) (drill 0.4) (layers F.Cu B.Cu) (net 10))
+  (via (at 59.055 53.975) (size 0.8) (drill 0.4) (layers F.Cu B.Cu) (net 10))
+  (via (at 57.785 53.975) (size 0.8) (drill 0.4) (layers F.Cu B.Cu) (net 10))
   (via (at 20.32 36.195) (size 0.8) (drill 0.4) (layers F.Cu B.Cu) (net 1))
   (via (at 20.32 37.465) (size 0.8) (drill 0.4) (layers F.Cu B.Cu) (net 1))
@@
   (via (at 48.26 49.53) (size 0.8) (drill 0.4) (layers F.Cu B.Cu) (net 2))
   (segment (start 49.8625 49.53) (end 48.26 49.53) (width 0.25) (layer F.Cu) (net 2))
-  (via (at 63.5 49.53) (size 0.8) (drill 0.4) (layers F.Cu B.Cu) (net 2))
-  (segment (start 63.5 49.53) (end 61.8 49.53) (width 0.25) (layer F.Cu) (net 2))
+  (via (at 61.595 49.53) (size 0.8) (drill 0.4) (layers F.Cu B.Cu) (net 2))
   (via (at 56.515 26.67) (size 0.8) (drill 0.4) (layers F.Cu B.Cu) (net 2))
   (segment (start 54.925 26.67) (end 56.515 26.67) (width 0.25) (layer F.Cu) (net 2))
@@
   (segment (start 84.885 58.625) (end 85.09 58.42) (width 0.25) (layer F.Cu) (net 2))
   (segment (start 84.885 60.96) (end 84.885 58.625) (width 0.25) (layer F.Cu) (net 2))
-  (via (at 59.055 51.435) (size 0.8) (drill 0.4) (layers F.Cu B.Cu) (net 10))
-  (via (at 57.785 51.435) (size 0.8) (drill 0.4) (layers F.Cu B.Cu) (net 10))
+  (segment (start 61.595 49.53) (end 63.07 49.53) (width 0.5) (layer F.Cu) (net 2))
+  (via (at 59.055 50.8) (size 0.8) (drill 0.4) (layers F.Cu B.Cu) (net 10))
+  (via (at 57.785 50.8) (size 0.8) (drill 0.4) (layers F.Cu B.Cu) (net 10))
   (segment (start 56.515 36.195) (end 55.88 35.56) (width 0.25) (layer F.Cu) (net 8))
   (segment (start 56.515 38.735) (end 56.515 36.195) (width 0.25) (layer F.Cu) (net 8))
@@
   (segment (start 56.515 46.355) (end 59.055 46.355) (width 0.5) (layer F.Cu) (net 10))
   (segment (start 58.85 46.56) (end 59.055 46.355) (width 0.25) (layer F.Cu) (net 10))
-  (segment (start 58.85 49.53) (end 58.85 46.56) (width 0.5) (layer F.Cu) (net 10))
   (segment (start 61.595 38.735) (end 61.595 41.275) (width 0.5) (layer F.Cu) (net 10))
   (segment (start 61.595 41.275) (end 59.055 43.815) (width 0.5) (layer F.Cu) (net 10))
@@
   (segment (start 59.5875 53.8725) (end 59.055 53.34) (width 0.25) (layer F.Cu) (net 10))
   (segment (start 60.12 53.34) (end 59.5875 53.8725) (width 0.5) (layer F.Cu) (net 10))
-  (segment (start 59.055 53.34) (end 57.785 53.34) (width 0.25) (layer B.Cu) (net 10))
-  (segment (start 57.785 53.34) (end 57.785 51.435) (width 0.25) (layer B.Cu) (net 10))
-  (segment (start 59.055 51.435) (end 59.055 53.34) (width 0.25) (layer B.Cu) (net 10))
-  (segment (start 57.785 51.435) (end 59.055 51.435) (width 0.5) (layer F.Cu) (net 10))
-  (segment (start 59.055 49.735) (end 58.85 49.53) (width 0.25) (layer F.Cu) (net 10))
-  (segment (start 59.055 51.435) (end 59.055 49.735) (width 0.5) (layer F.Cu) (net 10))
+  (segment (start 57.785 50.8) (end 59.055 50.8) (width 0.5) (layer F.Cu) (net 10))
+  (segment (start 59.055 48.465) (end 60.12 49.53) (width 0.5) (layer F.Cu) (net 10))
+  (segment (start 59.055 46.355) (end 59.055 48.465) (width 0.5) (layer F.Cu) (net 10))
+  (segment (start 57.785 51.435) (end 57.785 50.8) (width 0.25) (layer B.Cu) (net 10))
+  (segment (start 57.785 53.975) (end 57.785 51.435) (width 0.25) (layer B.Cu) (net 10))
+  (segment (start 59.055 51.435) (end 59.055 50.8) (width 0.25) (layer B.Cu) (net 10))
+  (segment (start 59.055 53.975) (end 59.055 51.435) (width 0.25) (layer B.Cu) (net 10))
+  (segment (start 60.12 49.735) (end 59.055 50.8) (width 0.5) (layer F.Cu) (net 10))
+  (segment (start 60.12 49.53) (end 60.12 49.735) (width 0.25) (layer F.Cu) (net 10))
   (segment (start 48.41 69.215) (end 41.91 69.215) (width 0.25) (layer F.Cu) (net 11))
   (segment (start 41.91 69.215) (end 38.735 69.215) (width 0.25) (layer F.Cu) (net 11))
@@
   (segment (start 28.575 30.1225) (end 28.575 33.3525) (width 0.25) (layer F.Cu) (net 16))
   (segment (start 51.7375 49.53) (end 54.3325 49.53) (width 0.25) (layer F.Cu) (net 17))
-  (segment (start 48.95 29.155) (end 48.95 22.755) (width 0.25) (layer F.Cu) (net 18))
-  (segment (start 46.355 31.75) (end 48.95 29.155) (width 0.25) (layer F.Cu) (net 18))
-  (segment (start 46.355 38.735) (end 46.355 31.75) (width 0.25) (layer F.Cu) (net 18))
+  (segment (start 46.355 31.75) (end 46.355 38.735) (width 0.25) (layer F.Cu) (net 18))
+  (segment (start 49.53 28.575) (end 46.355 31.75) (width 0.25) (layer F.Cu) (net 18))
+  (segment (start 49.53 27.94) (end 49.53 28.575) (width 0.25) (layer F.Cu) (net 18))
+  (segment (start 48.95 27.36) (end 49.53 27.94) (width 0.25) (layer F.Cu) (net 18))
+  (segment (start 48.95 22.755) (end 48.95 27.36) (width 0.25) (layer F.Cu) (net 18))
   (segment (start 48.895 38.735) (end 48.895 33.655) (width 0.25) (layer F.Cu) (net 19))
   (segment (start 48.895 33.655) (end 48.895 33.655) (width 0.25) (layer F.Cu) (net 19))
@@
   (segment (start 46.355 30.48) (end 46.355 30.48) (width 0.25) (layer B.Cu) (net 21))
   (via (at 46.355 30.48) (size 0.8) (drill 0.4) (layers F.Cu B.Cu) (net 21))
-  (segment (start 46.355 30.48) (end 46.355 24.765) (width 0.25) (layer F.Cu) (net 21))
-  (segment (start 45.95 22.755) (end 45.95 24.36) (width 0.25) (layer F.Cu) (net 21))
-  (segment (start 45.95 24.36) (end 46.355 24.765) (width 0.25) (layer F.Cu) (net 21))
+  (segment (start 45.95 30.075) (end 46.355 30.48) (width 0.25) (layer F.Cu) (net 21))
+  (segment (start 45.95 22.755) (end 45.95 30.075) (width 0.25) (layer F.Cu) (net 21))
   (segment (start 44.95 23.995) (end 44.95 22.755) (width 0.25) (layer F.Cu) (net 22))
   (segment (start 45.085 24.13) (end 44.95 23.995) (width 0.25) (layer F.Cu) (net 22))
@@
     (polygon
       (pts
-        (xy 21.59 35.56) (xy 21.59 57.15) (xy 19.05 59.69) (xy 19.05 66.675) (xy 17.78 67.945)
-        (xy 15.24 67.945) (xy 14.605 67.31) (xy 14.605 35.56) (xy 15.24 34.925) (xy 20.955 34.925)
+        (xy 21.59 35.56) (xy 21.59 57.15) (xy 19.05 59.69) (xy 19.05 67.31) (xy 18.415 67.945)
+        (xy 15.24 67.945) (xy 14.605 67.945) (xy 14.605 35.56) (xy 15.24 34.925) (xy 20.955 34.925)
       )
     )
@@
       (pts
         (xy 33.02 38.1) (xy 27.305 38.1) (xy 26.035 39.37) (xy 26.035 46.99) (xy 24.765 48.26)
-        (xy 24.13 48.26) (xy 20.955 45.085) (xy 24.13 41.91) (xy 24.13 38.735) (xy 26.035 36.83)
+        (xy 24.13 48.26) (xy 21.59 45.085) (xy 24.13 42.545) (xy 24.13 38.735) (xy 26.035 36.83)
         (xy 29.21 36.83) (xy 31.115 34.925) (xy 33.02 34.925)
       )
@@
     (polygon
       (pts
-        (xy 93.98 80.01) (xy 13.97 80.01) (xy 13.97 33.655) (xy 14.605 33.655) (xy 14.605 68.58)
-        (xy 17.78 68.58) (xy 19.685 66.675) (xy 19.685 60.325) (xy 22.225 57.785) (xy 22.225 33.655)
+        (xy 93.98 80.01) (xy 13.97 80.01) (xy 13.97 33.655) (xy 14.605 33.655) (xy 14.605 71.12)
+        (xy 17.78 71.12) (xy 19.685 69.215) (xy 19.685 60.325) (xy 22.225 57.785) (xy 22.225 33.655)
         (xy 15.24 33.655) (xy 13.97 32.385) (xy 13.97 13.97) (xy 93.98 13.97)
       )

Commit message: + logo
Parts:
- added REF**: KiCad-Logo2_5mm_SilkScreen, Symbol:KiCad-Logo2_5mm_SilkScreen, F.Cu at (34.9, 76.8)
- renumbered SW1 to Reset
Other:
- board text added: "Power"
- board text added: "System"

Commit message: minor fixes
Parts:
- moved   1.27 mm to (58.4, 20.3)
- moved   0.64 mm to (31.8, 70.5)
Routing:
- net VCC: track 204.2 -> 203.4 mm

Commit message: minor fixes
Parts:
- moved   1.27 mm to (33.0, 70.5)
Routing:
- net GND: vias 75 -> 78
Changed lines of the file:
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@@
     (thickness 1.6)
     (drawings 7)
-    (tracks 488)
+    (tracks 491)
     (zones 0)
     (modules 69)
@@
   )
   (module MountingHole:MountingHole_3.2mm_M3 (layer F.Cu)
-    (at 31.75 70.485)
+    (at 33.02 70.485)
     (descr "Mounting Hole 3.2mm, no annular, M3")
     (tags "mounting hole 3.2mm no annular m3")
@@
   (segment (start 84.885 60.96) (end 84.885 58.625) (width 0.25) (layer F.Cu) (net 2))
   (segment (start 61.595 49.53) (end 63.07 49.53) (width 0.5) (layer F.Cu) (net 2))
+  (via (at 31.75 48.26) (size 0.8) (drill 0.4) (layers F.Cu B.Cu) (net 2))
+  (via (at 31.75 46.99) (size 0.8) (drill 0.4) (layers F.Cu B.Cu) (net 2))
+  (via (at 31.75 52.07) (size 0.8) (drill 0.4) (layers F.Cu B.Cu) (net 2))
   (segment (start 56.515 36.195) (end 55.88 35.56) (width 0.25) (layer F.Cu) (net 8))
   (segment (start 56.515 38.735) (end 56.515 36.195) (width 0.25) (layer F.Cu) (net 8))
@@
       )
     )
+  )
+  (zone (net 36) (net_name AMP_IN) (layer F.Cu) (hatch edge 0.508)
+    (connect_pads (clearance 0.508))
+    (min_thickness 0.254)
+    (fill yes (arc_segments 32) (thermal_gap 0.508) (thermal_bridge_width 0.508))
+    (polygon
+      (pts
+        (xy 31.115 66.675) (xy 28.575 69.215) (xy 28.575 72.39) (xy 27.305 73.66) (xy 17.145 73.66)
+        (xy 16.51 73.025) (xy 16.51 71.755) (xy 17.145 71.12) (xy 18.415 71.12) (xy 24.13 65.405)
+        (xy 27.94 65.405) (xy 29.21 64.135) (xy 31.115 64.135)
+      )
+    )
+  )
+  (zone (net 36) (net_name AMP_IN) (layer F.Cu) (hatch edge 0.508)
+    (connect_pads (clearance 0.508))
+    (min_thickness 0.254)
+    (fill yes (arc_segments 32) (thermal_gap 0.508) (thermal_bridge_width 0.508))
+    (polygon
+      (pts
+        (xy 42.545 66.675) (xy 41.91 67.31) (xy 35.56 67.31) (xy 34.925 66.675) (xy 28.575 66.675)
+        (xy 28.575 64.77) (xy 29.21 64.135) (xy 29.21 62.23) (xy 29.845 61.595) (xy 42.545 61.595)
+      )
+    )
